File: docking_station/Hardware/docking_station.kicad_sch (KiCad schematic)
At the start: 81 parts, among them IC1 VOM1271T, IC2 VOM1271T, IC3 VOM1271T, IC4 VOM1271T, IC5 VOM1271T, J1 WAGO, J2 XT60, J3 Conn_01x05_Pin, J5 SUPPLY+, J6 SUPPLY-, K1 RELPOL R40N-3021-85-1024, Q1 SIDR392DP-T1-GE3, Q10 DN2540N8-G, Q11 DN2540N8-G, Q12 2N7002K, Q2 SIDR392DP-T1-GE3, Q3 SIDR392DP-T1-GE3, Q4 SIDR392DP-T1-GE3, Q5 SIDR392DP-T1-GE3, Q6 SIDR392DP-T1-GE3, Q7 SIDR392DP-T1-GE3, Q8 SIDR392DP-T1-GE3, Q9 SIDR392DP-T1-GE3, U1 LTC4357MS8, U2 ACS712xLCTR-20A, U3 L78L05AB, U4 LMV321IYLT, U5 MCP6561T-E/OT, U6 MCP6561T-E/OT

Commit message: trochę zmian fpt
Parts:
- removed TP23: TestPoint_2Pole, symbol Connector:TestPoint_2Pole
- added TP23, TP26: TestPoint, TestPoint:TestPoint_Bridge_Pitch3.81mm_Drill1.3mm, symbol Connector:TestPoint
- F1: footprint (none) -> firo_footprints:firo_fuse
Connections:
- net SENSE+: now also TP26.1
- net SENSE-: now also TP23.1
Changed lines of the file:
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@@
 	)
 	(junction
-		(at 153.67 137.16)
+		(at 31.75 137.16)
 		(diameter 0)
 		(color 0 0 0 0)
 	)
 	(junction
-		(at 157.48 68.58)
+		(at 153.67 137.16)
 		(diameter 0)
 		(color 0 0 0 0)
 	)
 	(junction
-		(at 223.52 102.87)
+		(at 157.48 68.58)
 		(diameter 0)
 		(color 0 0 0 0)
 	)
 	(junction
-		(at 33.02 137.16)
+		(at 223.52 102.87)
 		(diameter 0)
 		(color 0 0 0 0)
@@
 	)
 	(junction
-		(at 33.02 127)
-		(diameter 0)
-		(color 0 0 0 0)
-	)
-	(junction
 		(at 246.38 71.12)
 		(diameter 0)
@@
 		(color 0 0 0 0)
 	)
+	(junction
+		(at 31.75 127)
+		(diameter 0)
+		(color 0 0 0 0)
+	)
 	(wire
 		(pts
@@
 	(wire
 		(pts
-			(xy 29.21 137.16) (xy 33.02 137.16)
+			(xy 29.21 137.16) (xy 31.75 137.16)
 		)
 		(stroke
@@
 	(wire
 		(pts
-			(xy 29.21 127) (xy 33.02 127)
+			(xy 29.21 127) (xy 31.75 127)
 		)
 		(stroke
@@
 	(wire
 		(pts
-			(xy 33.02 137.16) (xy 34.29 137.16)
-		)
-		(stroke
-			(width 0)
-			(type default)
-		)
-	)
-	(wire
-		(pts
-			(xy 33.02 127) (xy 34.29 127)
-		)
-		(stroke
-			(width 0)
-			(type default)
-		)
-	)
-	(wire
-		(pts
 			(xy 256.54 55.88) (xy 246.38 55.88)
 		)
@@
 	(wire
 		(pts
+			(xy 31.75 137.16) (xy 34.29 137.16)
+		)
+		(stroke
+			(width 0)
+			(type default)
+		)
+	)
+	(wire
+		(pts
 			(xy 246.38 71.12) (xy 236.22 71.12)
 		)
@@
 	(wire
 		(pts
+			(xy 31.75 127) (xy 34.29 127)
+		)
+		(stroke
+			(width 0)
+			(type default)
+		)
+	)
+	(wire
+		(pts
 			(xy 128.27 132.08) (xy 133.35 132.08)
 		)
@@
 			)
 		)
-		(property "Footprint" ""
+		(property "Footprint" "firo_footprints:firo_fuse"
 			(at 49.53 46.228 90)
 			(effects
@@
 	)
 	(symbol
+		(lib_id "Connector:TestPoint")
+		(at 31.75 137.16 180)
+		(unit 1)
+		(exclude_from_sim no)
+		(in_bom yes)
+		(on_board yes)
+		(dnp no)
+		(property "Reference" "TP23"
+			(at 25.654 140.462 0)
+			(effects
+				(font
+					(size 1.27 1.27)
+				)
+				(justify right)
+			)
+		)
+		(property "Value" "TestPoint"
+			(at 28.194 146.05 0)
+			(effects
+				(font
+					(size 1.27 1.27)
+				)
+				(justify right)
+				(hide yes)
+			)
+		)
+		(property "Footprint" "TestPoint:TestPoint_Bridge_Pitch3.81mm_Drill1.3mm"
+			(at 26.67 137.16 0)
+			(effects
+				(font
+					(size 1.27 1.27)
+				)
+				(hide yes)
+			)
+		)
+		(property "Datasheet" "~"
+			(at 26.67 137.16 0)
+			(effects
+				(font
+					(size 1.27 1.27)
+				)
+				(hide yes)
+			)
+		)
+		(property "Description" "test point"
+			(at 31.75 137.16 0)
+			(effects
+				(font
+					(size 1.27 1.27)
+				)
+				(hide yes)
+			)
+		)
+		(pin "1"
+		)
+		(instances
+			(project "docking_station"
+				(path "/08748f9a-6084-44ea-8855-9d9812e8dfdd"
+					(reference "TP23")
+					(unit 1)
+				)
+			)
+		)
+	)
+	(symbol
 		(lib_id "Device:R_Small")
 		(at 57.15 148.59 270)
@@
 	)
 	(symbol
-		(lib_id "Connector:TestPoint_2Pole")
-		(at 33.02 132.08 270)
-		(mirror x)
-		(unit 1)
-		(exclude_from_sim no)
-		(in_bom yes)
-		(on_board yes)
-		(dnp no)
-		(property "Reference" "TP23"
-			(at 31.496 132.08 90)
-			(effects
-				(font
-					(size 1.27 1.27)
-				)
-				(justify right)
-			)
-		)
-		(property "Value" "TestPoint_2Pole"
-			(at 30.48 133.3499 90)
-			(effects
-				(font
-					(size 1.27 1.27)
-				)
-				(justify right)
-				(hide yes)
-			)
-		)
-		(property "Footprint" ""
-			(at 33.02 132.08 0)
-			(effects
-				(font
-					(size 1.27 1.27)
-				)
-				(hide yes)
-			)
-		)
-		(property "Datasheet" "~"
-			(at 33.02 132.08 0)
-			(effects
-				(font
-					(size 1.27 1.27)
-				)
-				(hide yes)
-			)
-		)
-		(property "Description" "2-polar test point"
-			(at 33.02 132.08 0)
-			(effects
-				(font
-					(size 1.27 1.27)
-				)
-				(hide yes)
-			)
-		)
-		(pin "2"
-		)
-		(pin "1"
-		)
-		(instances
-			(project "docking_station"
-				(path "/08748f9a-6084-44ea-8855-9d9812e8dfdd"
-					(reference "TP23")
-					(unit 1)
-				)
-			)
-		)
-	)
-	(symbol
 		(lib_id "power:+5V")
 		(at 68.58 123.19 0)
@@
 					(unit 1)
 				)
+			)
+		)
+	)
+	(symbol
+		(lib_id "Connector:TestPoint")
+		(at 31.75 127 0)
+		(unit 1)
+		(exclude_from_sim no)
+		(in_bom yes)
+		(on_board yes)
+		(dnp no)
+		(property "Reference" "TP26"
+			(at 30.734 123.698 0)
+			(effects
+				(font
+					(size 1.27 1.27)
+				)
+				(justify right)
+			)
+		)
+		(property "Value" "TestPoint"
+			(at 35.306 118.11 0)
+			(effects
+				(font
+					(size 1.27 1.27)
+				)
+				(justify right)
+				(hide yes)
+			)
+		)
+		(property "Footprint" "TestPoint:TestPoint_Bridge_Pitch3.81mm_Drill1.3mm"
+			(at 36.83 127 0)
+			(effects
+				(font
+					(size 1.27 1.27)
+				)
+				(hide yes)
+			)
+		)
+		(property "Datasheet" "~"
+			(at 36.83 127 0)
+			(effects
+				(font
+					(size 1.27 1.27)
+				)
+				(hide yes)
+			)
+		)
+		(property "Description" "test point"
+			(at 31.75 127 0)
+			(effects
+				(font
+					(size 1.27 1.27)
+				)
+				(hide yes)
+			)
+		)
+		(pin "1"
+		)
+		(instances
+			(project "docking_station"
+				(path "/08748f9a-6084-44ea-8855-9d9812e8dfdd"
+					(reference "TP26")
+					(unit 1)
+				)

Commit message: introductory compontent layout
grouped the components, prepped the group layout. The board does seem doable
Parts:
- removed U5, U6: MCP6561T-E/OT, Package_TO_SOT_SMD:SOT-23-5, symbol Comparator:LM397
- added U5, U6: MCP6561T-E/OT, Package_TO_SOT_SMD:SOT-23-5, symbol Comparator:MCP6561-OT
- J5, J6: footprint (none) -> firo_footprints:14 AWG soldering pad
- Q1, Q2, Q3, Q4, Q5, Q6, Q7, Q8, Q9: footprint Package_SO:PowerPAK_SO-8_Single -> firo_footprints:PowerPAK_SO-8DC for VISHAY SIDR392DP-T1-GE3
- TP23, TP24, TP25, TP26: footprint TestPoint:TestPoint_Bridge_Pitch3.81mm_Drill1.3mm -> TestPoint:TestPoint_Pad_D2.0mm
- U4: footprint Package_TO_SOT_SMD:SOT-23 -> Package_TO_SOT_SMD:SOT-23-5
Connections:
- net +5V: now also U4.5 (V+), U5.5 (V+), U6.5 (V+); no longer U4.3 (V+)
- net AMP_OUT: now also U4.4, U5.4 (-); no longer U4.5
- net GND: now also U4.2 (V-), U5.2 (V-), U6.2 (V-); no longer U4.4 (V-)
- net at C7.1, R7.1, R8.1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: now also U6.3 (+)
- net at JP1.1 (A), R10.2, TP9.1: now also U6.1
- net at R4.1, R5.1: now also U4.3 (-); no longer U4.2 (-)
- net at R7.2, TP7.1: now also U5.1
- net at R10.1, RV2.2: now also U6.4 (-)
- net at RV1.2: now also U5.3 (+)
Other:
- note added: "PC FAN CONNECTOR?"

Commit message: big layout progress
Parts:
- added J4: SUPPLY+, firo_footprints:14 AWG soldering pad, symbol Connector:Conn_01x01_Pin
- added J7: SUPPLY-, firo_footprints:14 AWG soldering pad, symbol Connector:Conn_01x01_Pin
Connections:
- net VDC is gone; now on net +24V: Q2.3 (D), Q6.3 (D)
- net GND: now also J7.1 (Pin_1)
- net CS_3: now reaches IC3.3 (K_2), Q6.1 (S), Q7.1 (S), TP17.1
- net CS_4: now reaches IC4.3 (K_2), Q8.1 (S), Q9.1 (S), TP18.1
- net CS_2: now reaches IC2.3 (K_2), Q4.1 (S), Q5.1 (S), TP16.1
- net at F1.1, J5.1 (Pin_1), TP19.1: now also J4.1 (Pin_1)
- net CS_1: now reaches IC1.3 (K_2), Q2.1 (S), Q3.1 (S), TP15.1
