File: docking_station/Hardware/docking_station.kicad_pcb (KiCad board)
At the start: 2 copper layers, 115 x 43 mm, 108 parts, among them IC1 VOM1271T, IC2 VOM1271T, IC3 VOM1271T, IC4 VOM1271T, IC5 VOM1271T, J1 SUPPLY+, J2 SUPPLY-, J3 Conn_01x05_Pin, J4 XT60, J5 WAGO, K1 RELPOL R40N-3021-85-1024, Q1 SIDR392DP-T1-GE3, Q10 2N7002K, Q11 2N7002K, Q12 2N7002K, Q13 2N7002K, Q2 SIDR392DP-T1-GE3, Q3 SIDR392DP-T1-GE3, Q4 SIDR392DP-T1-GE3, Q5 SIDR392DP-T1-GE3, Q6 SIDR392DP-T1-GE3, Q7 SIDR392DP-T1-GE3, Q8 SIDR392DP-T1-GE3, Q9 SIDR392DP-T1-GE3, U1 LTC4357MS8, U2 L78L05AB, U3 ACS712xLCTR-20A, U4 LMV321IYLT, U5 MCP6561T-E/OT, U6 MCP6561T-E/OT, U7 MCP6561T-E/OT

Commit message: gaining_a_level_of_exhaustion_xd
Routing:
- net SENSE-: track 4.35 -> 4.91 mm
Changed lines of the file:
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@@
 	)
 	(via
-		(at 159.751712 98.725856)
+		(at 159.854421 98.748132)
 		(size 0.7)
 		(drill 0.3)
@@
 		(start 155.2 107.8)
 		(end 155.5 107.5)
-		(width 0.2)
+		(width 0.254)
 		(layer "F.Cu")
 		(net 3)
@@
 		(start 155.5 107.5)
 		(end 160.1 107.5)
-		(width 0.2)
+		(width 0.254)
 		(layer "F.Cu")
 		(net 3)
@@
 	)
 	(segment
-		(start 155.2 107.8)
-		(end 155.5875 107.8)
-		(width 0.127)
-		(layer "B.Cu")
-		(net 3)
-	)
-	(segment
 		(start 145.41 99)
 		(end 145.41 99.747948)
@@
 	)
 	(segment
-		(start 158.6 100)
-		(end 158.6 102)
-		(width 0.127)
+		(start 159.165 102.565)
+		(end 159.73 102.565)
+		(width 0.254)
 		(layer "B.Cu")
 		(net 31)
 	)
 	(segment
-		(start 158.275 99.675)
-		(end 158.6 100)
-		(width 0.127)
+		(start 158.496 99.896)
+		(end 158.496 101.896)
+		(width 0.254)
 		(layer "B.Cu")
 		(net 31)
 	)
 	(segment
-		(start 158.6 102)
-		(end 159.165 102.565)
-		(width 0.127)
+		(start 157.1875 99.675)
+		(end 158.275 99.675)
+		(width 0.254)
 		(layer "B.Cu")
 		(net 31)
 	)
 	(segment
-		(start 157.1875 99.675)
-		(end 158.275 99.675)
-		(width 0.127)
+		(start 158.275 99.675)
+		(end 158.496 99.896)
+		(width 0.254)
 		(layer "B.Cu")
 		(net 31)
 	)
 	(segment
-		(start 158.927 100.827)
-		(end 159.395 101.295)
-		(width 0.127)
+		(start 158.496 101.896)
+		(end 159.165 102.565)
+		(width 0.254)
 		(layer "B.Cu")
-		(net 32)
+		(net 31)
 	)
 	(segment
-		(start 157.1875 97.725)
-		(end 158.025 97.725)
-		(width 0.127)
+		(start 159.395 101.295)
+		(end 159.73 101.295)
+		(width 0.254)
 		(layer "B.Cu")
 		(net 32)
 	)
 	(segment
-		(start 159.395 101.295)
-		(end 159.73 101.295)
-		(width 0.127)
+		(start 159.0572 98.7572)
+		(end 159.0572 100.9572)
+		(width 0.254)
 		(layer "B.Cu")
 		(net 32)
@@
 	(segment
 		(start 158.025 97.725)
-		(end 158.927 98.627)
-		(width 0.127)
+		(end 159.0572 98.7572)
+		(width 0.254)
+		(layer "B.Cu")
+		(net 32)
+	)
+	(segment
+		(start 159.0572 100.9572)
+		(end 159.395 101.295)
+		(width 0.254)
 		(layer "B.Cu")
 		(net 32)
 	)
 	(segment
-		(start 158.927 98.627)
-		(end 158.927 100.827)
-		(width 0.127)
+		(start 157.1875 97.725)
+		(end 158.025 97.725)
+		(width 0.254)
 		(layer "B.Cu")
 		(net 32)

Commit message: last commit before gerber export
Other:
- board text added: "CHECK SUPPLY POLARITY"
- board text added: "PAD CONNECTOR"
Changed lines of the file:
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@@
 		(tags "RC Connector XT60")
 		(property "Reference" "J4"
-			(at -3.6 -16.5 -90)
+			(at -3.6 -16.5 90)
 			(layer "F.SilkS")
 			(hide yes)
@@
 		)
 		(property "Value" "XT60"
-			(at -3.6 4 -90)
+			(at -3.6 4 90)
 			(layer "F.Fab")
 			(effects
@@
 			(layer "F.Fab")
 		)
-		(fp_text user "-"
-			(at -0.7 3.05 -90)
-			(layer "F.SilkS")
-			(effects
-				(font
-					(size 1 1)
-					(thickness 0.15)
-				)
-			)
-		)
-		(fp_text user "+"
-			(at -6.3 3.15 -90)
-			(layer "F.SilkS")
-			(effects
-				(font
-					(size 1.5 1.5)
-					(thickness 0.15)
-				)
-			)
-		)
 		(fp_text user "${REFERENCE}"
-			(at -3.6 -3.6 -90)
+			(at -3.6 -3.6 90)
 			(layer "F.Fab")
 			(effects
@@
 		)
 	)
+	(gr_text "CHECK SUPPLY POLARITY"
+		(at 152.527 124.333 0)
+		(layer "F.SilkS" knockout)
+		(effects
+			(font
+				(size 1.5 1.5)
+				(thickness 0.25)
+				(bold yes)
+			)
+			(justify left bottom)
+		)
+	)
 	(gr_text "T PROBE"
 		(at 158.5 105.3 0)
@@
 	)
 	(gr_text "SUPPLY-"
-		(at 181.2 123.3 0)
+		(at 181.737 123.3 0)
 		(layer "F.SilkS")
 		(effects
@@
 			)
 			(justify left bottom)
+		)
+	)
+	(gr_text "PAD CONNECTOR"
+		(at 182.710664 109.428933 90)
+		(layer "F.SilkS" knockout)
+		(effects
+			(font
+				(size 1 1)
+				(thickness 0.2)
+				(bold yes)
+			)
+			(justify left bottom)

Commit message: shopping list, gerbers and board updates
Other:
- board text added: "JLCJLCJLCJLC"
Changed lines of the file:
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@@
 		(allow_soldermask_bridges_in_footprints no)
 		(pcbplotparams
-			(layerselection 0x0001020_7fffffff)
+			(layerselection 0x00010fc_ffffffff)
 			(plot_on_all_layers_selection 0x0000000_00000000)
 			(disableapertmacros no)
-			(usegerberextensions no)
-			(usegerberattributes yes)
-			(usegerberadvancedattributes yes)
-			(creategerberjobfile yes)
+			(usegerberextensions yes)
+			(usegerberattributes no)
+			(usegerberadvancedattributes no)
+			(creategerberjobfile no)
 			(dashed_line_dash_ratio 12.000000)
 			(dashed_line_gap_ratio 3.000000)
 			(svgprecision 4)
 			(plotframeref no)
-			(viasonmask yes)
+			(viasonmask no)
 			(mode 1)
 			(useauxorigin no)
@@
 			(psnegative no)
 			(psa4output no)
-			(plotreference no)
+			(plotreference yes)
 			(plotvalue no)
-			(plotfptext no)
+			(plotfptext yes)
 			(plotinvisibletext no)
 			(sketchpadsonfab no)
-			(subtractmaskfromsilk no)
-			(outputformat 3)
+			(subtractmaskfromsilk yes)
+			(outputformat 1)
 			(mirror no)
 			(drillshape 0)
 			(scaleselection 1)
-			(outputdirectory "")
+			(outputdirectory "gerber/")
 		)
 	)
@@
 	)
 	(gr_text "CHECK SUPPLY POLARITY"
-		(at 152.527 124.333 0)
+		(at 155 124.3 0)
 		(layer "F.SilkS" knockout)
 		(effects
 			(font
-				(size 1.5 1.5)
+				(size 1.5 1.35)
 				(thickness 0.25)
 				(bold yes)
@@
 	)
 	(gr_text "SUPPLY-"
-		(at 181.737 123.3 0)
+		(at 181.3 123.3 0)
 		(layer "F.SilkS")
 		(effects
@@
 		(layer "F.SilkS")
 		(effects
+			(font
+				(size 1 1)
+				(thickness 0.15)
+			)
+			(justify left bottom)
+		)
+	)
+	(gr_text "JLCJLCJLCJLC"
+		(at 131.2 109.3 90)
+		(layer "F.SilkS")
+		(effects
