File: charging_controller/Hardware/charging_controller.kicad_sch (KiCad schematic)
At the start: 30 parts, among them J1 XT60, J2 XT60, J3 ??, J4 Conn_01x08_Pin, Q1 PMOS, Q2 NMOS, SW1 SW_Push, U1 STM32F103CBTx, U2 MAX5035AUSA, U3 ACS712xLCTR-20A

Commit message: i_hate_git_please_end_this
Parts:
- removed C10: 100nF, symbol Device:C_Small
- removed C11: 35SVT39M, symbol Device:C_Polarized_Small
- removed D2: STPS1L30U, symbol Device:D_Schottky_Small
- removed L1: MURATA 1433445C 300uH, symbol Device:L_Small
- removed U2: MAX5035AUSA, Package_SO:SOIC-8_3.9x4.9mm_P1.27mm, symbol Regulator_Switching:MAX5035AUSA
- added J10: CAN, symbol Connector_Generic:Conn_02x02_Odd_Even
- added J11: HALL1, symbol Connector:Conn_01x03_Pin
- added J12: HALL2, symbol Connector:Conn_01x03_Pin
- added J5, J6, J8, J9: Conn_01x01, symbol Connector_Generic:Conn_01x01
- added J7: BAT_CONN, symbol Connector:Conn_01x02_Pin
- added M1: Motor_DC, symbol Motor:Motor_DC
- added U2: NCP114AMX330TBG, Package_SO:TSOP-5_1.65x3.05mm_P0.95mm, symbol Regulator_Linear:NCP1117-1.5_SOT223
- C9: footprint (none) -> Capacitor_SMD:C_0805_2012Metric
- R2: value 110k -> 1k
- R4: value 270k -> 1k
Connections:
- net +24V: now also J8.1 (Pin_1); no longer R4.1
- net GND: now also C9.2, J10.1 (Pin_1), J11.2 (Pin_2), J12.2 (Pin_2), J9.1 (Pin_1); no longer R2.2
- net +5V: now reaches R2.1
- net +5V: now also C9.1, R4.1, U3.8 (VCC), J10.4 (Pin_4), J11.1 (Pin_1), J12.1 (Pin_1); no longer R4.2
- new net: J6.1 (Pin_1), J7.2 (Pin_2)
- new net: J5.1 (Pin_1), J7.1 (Pin_1)
- new net CAN+: J10.3 (Pin_3)
- new net CAN-: J10.2 (Pin_2)
- new net HALL1: J11.3 (Pin_3), R2.2
- new net HALL2: J12.3 (Pin_3), R4.2
- no-connect marks 0 -> 1
Other:
- note added: "Opt. batt volt. converter"
- moved on the sheet: C8, JP1, R3, SW1, U1

Commit message: update
Parts:
- removed U2: NCP114AMX330TBG, Package_SO:TSOP-5_1.65x3.05mm_P0.95mm, symbol Regulator_Linear:NCP1117-1.5_SOT223
Other:
- moved on the sheet: J10, J11, J12, J4, R2, R4

Commit message: small changes
Parts:
- added C10: 4.7uF, symbol Device:C_Small
- added C11: 1uF, symbol Device:C_Small
- added D2: 3V3, symbol Device:D_Zener
- added R5, R6: R, symbol Device:R
- added R7: ??, symbol Device:R
- added TH1, TH2: Thermistor, symbol Device:Thermistor
- added U2: NCP114BSN330T1G, Package_SO:TSOP-5_1.65x3.05mm_P0.95mm, symbol FIRO_collected:ONESMI NCP114BSN330T1G
Connections:
- net +3V3: now also C11.1, R5.1, R6.1, U2.5 (VO)
- net +5V: now also C10.1, U2.1 (VI), U2.3 (EN)
- net GND: now also C10.2, C11.2, D2.2 (A), TH1.2, TH2.2, U2.2 (GND)
- net JNTRST: now also U1.40 (PB4)
- net JTCK/SWCLK: now also U1.37 (PA14)
- net JTDI: now also U1.38 (PA15)
- net JTDO/TRACESWO: now also U1.39 (PB3)
- net JTMS/SWDIO: now also U1.34 (PA13)
- net at J1.1 (Pin_1), Q2.3 (S), U3.1 (IP+)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: now also R7.1
- new net SENSE: D2.1 (K), R7.2
- new net T1: R5.2, TH1.1
- new net T2: R6.2, TH2.1
Other:
- note added: "A_IN"
- note added: "D_IN"
- note added: "HIGH - no magnet"
- note added: "OUTPUT"
- moved on the sheet: C12, C9, J1, J3, J5, J6, J7, J8, J9, Q2, U3

Commit message: handoff_to_office
Parts:
- removed M1: Motor_DC, symbol Motor:Motor_DC
- removed Q1: PMOS, symbol Simulation_SPICE:PMOS
- removed R3: R_Small, symbol Device:R_Small
- added C13, C14: 100nF, Capacitor_SMD:C_0805_2012Metric, symbol Device:C_Small
- added D3: D, symbol Device:D
- added JP2, JP3, JP4: SolderJumper_3_Bridged12, Jumper:SolderJumper-3_P1.3mm_Bridged12_RoundedPad1.0x1.5mm, symbol Jumper:SolderJumper_3_Bridged12
- added Q3: STD36P4LLF6, Package_TO_SOT_SMD:TO-252-2, symbol Device:Q_PMOS_GDS
- added R10: 120, symbol Device:R_Small
- added R8, R9: 10k, symbol Device:R_Small
- added U4: MCP2562-E-SN, Package_SO:SOIC-8_3.9x4.9mm_P1.27mm, symbol Interface_CAN_LIN:MCP2562-E-SN
- added U5: L6201PS, Package_SO:HSOP-20-1EP_11.0x15.9mm_P1.27mm_SlugDown, symbol FIRO_collected:L6201PS
- C1, C10, C11, C2, C3, C4, C5, C6, C7: footprint (none) -> Capacitor_SMD:C_0805_2012Metric
- C8: value C_Small -> 100nF; footprint (none) -> Capacitor_SMD:C_0805_2012Metric
- D1: value gate satefy -> 5V
- J1, J2: footprint (none) -> firo_footprints:AMASS_XT60PW-F-MP
- J10: footprint (none) -> Connector_TE-Connectivity:TE_Micro-MaTch_215079-4_2x02_P1.27mm_Vertical
- J4: footprint (none) -> Connector_PinHeader_2.54mm:PinHeader_2x08_P2.54mm_Vertical
- R1: value diode current -> 22k
Connections:
- net +24V: now also Q3.3 (S)
- net +3V3: now also JP3.1 (A), R8.2
- net +5V: now also C13.2, JP3.3 (B), U4.3 (VDD)
- net CAN+: now also R10.1, U4.7 (CANH)
- net CAN-: now also R10.2, U4.6 (CANL)
- net GND: now also C8.2, C13.1, C14.1, JP4.1 (A), R9.1, U4.2 (VSS)
- net at J1.1 (Pin_1), R7.1, U3.1 (IP+)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: now also D3.1 (K); no longer Q2.3 (S)
- net BOOT1: now reaches U1.20 (PB2)
- net at U1.44 (BOOT0): now also JP2.2 (C)
- net at J2.1 (Pin_1): now also Q3.2 (D)
- net at D1.2 (A), R1.1: now also Q3.1 (G)
- new net: JP2.1 (A), R9.2
- new net: JP2.3 (B), R8.1
- new net: JP4.2 (C), U4.8 (STBY)
- new net: D3.2 (A), Q2.3 (S)
- new net: C14.2, JP3.2 (C), U4.5 (Vio)
- new net: U5.1 (GND), U5.10 (GND)
- new net: U5.11 (GND), U5.20 (GND)
- new net CANRX: U4.4 (RXD)
- new net CANSTBY: JP4.3 (B)
- new net CANTX: U4.1 (TXD)
Other:
- note added: "BOOT0 jumper"
- note added: "NRST button"
- note added: "Opt. 42V to 5V converter"
- note removed: "Opt. batt volt. converter"
- moved on the sheet: C1, C10, C11, C12, C2, C3, C4, C5, C6, C7, C8, C9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

Commit message: a lot of work done
Parts:
- removed D3: D, symbol Device:D
- removed J7: BAT_CONN, symbol Connector:Conn_01x02_Pin
- removed Q2: NMOS, symbol Simulation_SPICE:NMOS
- removed U5: L6201PS, Package_SO:HSOP-20-1EP_11.0x15.9mm_P1.27mm_SlugDown, symbol FIRO_collected:L6201PS
- added D4: DST5100S, Package_TO_SOT_SMD:TO-277B, symbol Device:D_Schottky_AAK
- added F1: Fuse_Small, symbol Device:Fuse_Small
- added H1, H2, H3, H4: MountingHole_Pad, MountingHole:MountingHole_3.2mm_M3_Pad_Via, symbol Mechanical:MountingHole_Pad
- added J13: B2B, Connector_PinHeader_2.54mm:PinHeader_2x08_P2.54mm_Vertical, symbol Connector_Generic:Conn_02x08_Odd_Even
- added J7: XT60, Connector_AMASS:AMASS_XT60-F_1x02_P7.20mm_Vertical, symbol Connector_Generic_MountingPin:Conn_01x02_MountingPin
- added Q1: 2N7002K, Package_TO_SOT_SMD:SOT-23, symbol Transistor_FET:2N7002K
- added R11, R3: Trim, Resistor_SMD:R_0603_1608Metric, symbol Device:R_Small
- added R12: ??, Resistor_SMD:R_0402_1005Metric, symbol Device:R
- added R13: R, Resistor_SMD:R_0402_1005Metric, symbol Device:R
- added U5: THN 20WIR, firo_footprints:TRACO THN 20WIR, symbol FIRO_collected:TRACO_THN20WIR
- C1, C13, C14, C2, C3, C4, C5, C7, C8, C9: footprint Capacitor_SMD:C_0805_2012Metric -> Capacitor_SMD:C_0402_1005Metric
- D1, D2: footprint (none) -> Diode_SMD:D_SOD-123
- J1: value XT60 -> XT30; footprint firo_footprints:AMASS_XT60PW-F-MP -> Connector_AMASS:AMASS_XT30PW-M_1x02_P2.50mm_Horizontal
- J3: value ?? -> XT30; footprint (none) -> Connector_AMASS:AMASS_XT30PW-F_1x02_P2.50mm_Horizontal
- J4: footprint Connector_PinHeader_2.54mm:PinHeader_2x08_P2.54mm_Vertical -> Connector_PinHeader_2.54mm:PinHeader_2x04_P2.54mm_Vertical
- JP1: footprint (none) -> Jumper:SolderJumper-2_P1.3mm_Bridged_RoundedPad1.0x1.5mm
- Q3: value STD36P4LLF6 -> DMP6023LE-13; footprint Package_TO_SOT_SMD:TO-252-2 -> Package_TO_SOT_SMD:SOT-223-3_TabPin2
- R1: value 22k -> ??; footprint (none) -> Resistor_SMD:R_0603_1608Metric
- R10: footprint (none) -> Resistor_SMD:R_0805_2012Metric
- R2, R4: footprint (none) -> Resistor_SMD:R_0603_1608Metric
- R5, R6, R7, R8, R9: footprint (none) -> Resistor_SMD:R_0402_1005Metric
- SW1: footprint (none) -> Button_Switch_SMD:SW_SPST_EVQP7C
- TH1: value Thermistor -> PAD_TH
- TH2: value Thermistor -> Board_TH; footprint (none) -> Resistor_SMD:R_0603_1608Metric
Connections:
- net +24V: now also Q1.3 (D), R3.1, U5.4 (+Vout); no longer D1.1 (K), J8.1 (Pin_1), Q3.3 (S)
- net +3V3: now also J13.9 (Pin_9), R13.2
- net +5V: now also J8.1 (Pin_1), J13.1 (Pin_1)
- net CHG_INIT: now also Q1.1 (G)
- net GND: now also J1.1 (Pin_1), J2.1 (Pin_1), J3.1 (Pin_1), J6.1 (Pin_1), H1.1, H2.1, H3.1, H4.1, J13.16 (Pin_16), J7.1 (Pin_1), J7.MP (MountPin), R11.2, R12.2, U5.2 (-Vin), U5.6 (-Vout); no longer J1.2 (Pin_2), J2.2 (Pin_2), J3.2 (Pin_2)
- net SENSE: now also R12.1
- net at U3.1 (IP+), U3.2 (IP+): now also J3.2 (Pin_2), D4.3 (K); no longer J1.1 (Pin_1), R7.1
- net at U3.3 (IP-), U3.4 (IP-): now also J1.2 (Pin_2), R7.1; no longer J3.1 (Pin_1)
- net BOOT0: now reaches JP2.2 (C), U1.44 (BOOT0)
- net at Q3.2 (D): now also J2.2 (Pin_2), J7.2 (Pin_2); no longer J2.1 (Pin_1)
- net +BATT: now reaches J5.1 (Pin_1)
- net +BATT: now also F1.2, U5.1 (+Vin)
- new net: D4.1 (A), D4.2 (A), Q1.2 (S)
- new net: R11.1, R3.2, U5.5 (Trim)
- new net: D1.1 (K), F1.1, Q3.3 (S)
- new net IN1: J13.2 (Pin_2)
- new net IN2: J13.4 (Pin_4)
- new net MOT_EN: J13.6 (Pin_6)
- new net T3: J13.12 (Pin_12), R13.1
Other:
- note added: "ADR5043?"
- note added: "BAT to 24V converter"
- note added: "BAT_CONN"
- note added: "To PAD"
- note added: "closing mosfet"
- note removed: "24V in"
- note removed: "Pad conn"
- moved on the sheet: C12, C13, C9, D1, D2, J1, J11, J2, J3, J5, J6, J8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

Commit message: gaining_a_level_of_exhaustion_xd
Parts:
- removed F1: Fuse_Small, symbol Device:Fuse_Small
- removed J11: HALL1, symbol Connector:Conn_01x03_Pin
- removed J12: HALL2, symbol Connector:Conn_01x03_Pin
- removed TH1: PAD_TH, symbol Device:Thermistor
- added J11, J14: HALL2, firo_footprints:TEConnectivity_RITS_Header_3P_V, symbol Connector_Generic_MountingPin:Conn_01x03_MountingPin
- added J12: Pad_TH, firo_footprints:TEConnectivity_RITS_Header_3P_V, symbol Connector_Generic_MountingPin:Conn_01x03_MountingPin
- added JP5: Jumper_2_Small_Open, Jumper:SolderJumper-2_P1.3mm_Open_RoundedPad1.0x1.5mm, symbol Jumper:Jumper_2_Small_Open
Connections:
- net +5V: now also J11.1 (Pin_1), J14.1 (Pin_1)
- net +BATT: now also D1.1 (K), Q3.3 (S)
- net BOOT1: now also J13.14 (Pin_14)
- net CANRX: now also U1.32 (PA11)
- net CANSTBY: now also U1.28 (PB15)
- net CANTX: now also U1.31 (PA10)
- net CHG_CURR: now also U1.18 (PB0)
- net CHG_INIT: now also U1.15 (PA5)
- net GND: now also J13.15 (Pin_15), J13.7 (Pin_7), J11.2 (Pin_2), J11.MP (MountPin), J12.2 (Pin_2), J12.3 (Pin_3), J12.MP (MountPin), J14.2 (Pin_2), J14.MP (MountPin), JP5.2 (B); no longer J10.1 (Pin_1)
- net HALL1: now also U1.26 (PB13), J11.3 (Pin_3)
- net HALL2: now also U1.27 (PB14), J14.3 (Pin_3)
- net IN1: now also U1.46 (PB9)
- net IN2: now also U1.45 (PB8)
- net MOT_EN: now also U1.43 (PB7)
- net SENSE: now also U1.25 (PB12)
- net T1: now also U1.19 (PB1), J12.1 (Pin_1)
- net T2: now also U1.17 (PA7)
- net T3: now also U1.16 (PA6)
- net A8: now reaches U1.12 (PA2)
- net A8: now also J13.8 (Pin_8)
- net A5: now reaches U1.13 (PA3)
- net A5: now also J13.5 (Pin_5)
- net A10: now reaches U1.14 (PA4)
- net A10: now also J13.10 (Pin_10)
- net ROn/Off: now reaches U5.3 (ROn/Off)
- new net: J10.1 (Pin_1), JP5.1 (A)
- no-connect marks 1 -> 3
Other:
- note removed: "A_IN"
- note removed: "D_IN"
- moved on the sheet: R5

Commit message: PCBs possibly finished + some file org
Parts:
- removed J5, J6, J8, J9: Conn_01x01, symbol Connector_Generic:Conn_01x01
- added D3, D5, D6: G2V4, LED_SMD:LED_0805_2012Metric, symbol Device:LED
- added D7, D8: B3V1, LED_SMD:LED_0805_2012Metric, symbol Device:LED
- added IC1: VOM1271T, firo_footprints:SOP254P675X240-4N, symbol VOM1271T:VOM1271T
- added R14: 120, Resistor_SMD:R_0402_1005Metric, symbol Device:R
- added R15: 2k2, Resistor_SMD:R_1206_3216Metric, symbol Device:R
- added R16: 240, Resistor_SMD:R_0805_2012Metric, symbol Device:R
- added R17: 120, Resistor_SMD:R_0805_2012Metric, symbol Device:R
- added R18, R19: 20, Resistor_SMD:R_0805_2012Metric, symbol Device:R
- D1: value 5V -> 10V
- R1: value ?? -> 47k
Connections:
- net +24V: now also R15.1
- net +3V3: now also R17.1
- net +5V: now also R16.1
- net CHG_INIT: now also R14.1; no longer Q1.1 (G)
- net GND: now also D3.1 (K), D5.1 (K), D6.1 (K), D7.1 (K), D8.1 (K), IC1.2 (K_1)
- net D2: now reaches U1.4 (PC15)
- net D2: now also R18.1
- net D1: now reaches U1.5 (PD0)
- net D1: now also R19.1
- net at D4.1 (A), D4.2 (A), Q1.2 (S): now also IC1.3 (K_2)
- new net: D3.2 (A), R15.2
- new net: D8.2 (A), R19.2
- new net: IC1.1 (A_1), R14.2
- new net: D7.2 (A), R18.2
- new net: D5.2 (A), R16.2
- new net: IC1.4 (A_2), Q1.1 (G)
- new net: D6.2 (A), R17.2
Other:
- note added: "Turn off circuit??"
- note removed: "ADR5043?"
- note removed: "OUTPUT"
- note removed: "Opt. 42V to 5V converter"
- note removed: "closing mosfet"
- title: (none) -> Charging controller for FIRO 2.1 rover - main board
- moved on the sheet: C12, C9, D1, D2, D4, H1, H2, H3, H4, J1, J10, J11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

Commit message: a lot of work - charging main BOM complete
Parts:
- C4: footprint Capacitor_SMD:C_0402_1005Metric -> Capacitor_SMD:C_0805_2012Metric
- D1: footprint Diode_SMD:D_SOD-123 -> Diode_SMD:D_SOD-128
- D2: footprint Diode_SMD:D_SOD-123 -> Diode_SMD:D_SOD-523
- R1: value 47k -> 39k
- R12: value ?? -> 6k8
- R13, R5, R6: value R -> 5k6
- R14: footprint Resistor_SMD:R_0402_1005Metric -> Resistor_SMD:R_0805_2012Metric
- R2, R4: footprint Resistor_SMD:R_0603_1608Metric -> Resistor_SMD:R_0402_1005Metric
- R7: value ?? -> 39k; footprint Resistor_SMD:R_0402_1005Metric -> Resistor_SMD:R_0603_1608Metric
Changed lines of the file:
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@@
 			)
 		)
-		(property "Footprint" "Resistor_SMD:R_0603_1608Metric"
+		(property "Footprint" "Resistor_SMD:R_0402_1005Metric"
 			(at 38.1 177.8 0)
 			(effects
@@
 			)
 		)
-		(property "Value" "R"
+		(property "Value" "5k6"
 			(at 269.24 119.3801 0)
 			(effects
@@
 			)
 		)
-		(property "Footprint" "Resistor_SMD:R_0402_1005Metric"
+		(property "Footprint" "Resistor_SMD:R_0805_2012Metric"
 			(at 99.822 86.36 90)
 			(effects
@@
 			)
 		)
-		(property "Value" "??"
+		(property "Value" "6k8"
 			(at 41.91 126.9999 0)
 			(effects
@@
 			)
 		)
-		(property "Footprint" "Resistor_SMD:R_0603_1608Metric"
+		(property "Footprint" "Resistor_SMD:R_0402_1005Metric"
 			(at 38.1 158.75 0)
 			(effects
@@
 			)
 		)
-		(property "Value" "??"
+		(property "Value" "39k"
 			(at 36.83 118.1099 0)
 			(effects
@@
 			)
 		)
-		(property "Footprint" "Resistor_SMD:R_0402_1005Metric"
+		(property "Footprint" "Resistor_SMD:R_0603_1608Metric"
 			(at 32.512 116.84 90)
 			(effects
@@
 			)
 		)
-		(property "Footprint" "Capacitor_SMD:C_0402_1005Metric"
+		(property "Footprint" "Capacitor_SMD:C_0805_2012Metric"
 			(at 201.93 59.69 0)
 			(effects
@@
 			)
 		)
-		(property "Value" "R"
+		(property "Value" "5k6"
 			(at 76.2 165.0999 0)
 			(effects
@@
 			)
 		)
-		(property "Footprint" "Diode_SMD:D_SOD-123"
+		(property "Footprint" "Diode_SMD:D_SOD-523"
 			(at 34.29 125.73 0)
 			(effects
@@
 			)
 		)
-		(property "Value" "47k"
+		(property "Value" "39k"
 			(at 44.45 44.4499 0)
 			(effects
@@
 			)
 		)
-		(property "Value" "R"
+		(property "Value" "5k6"
 			(at 99.06 165.0999 0)
 			(effects
@@
 			)
 		)
-		(property "Footprint" "Diode_SMD:D_SOD-123"
+		(property "Footprint" "Diode_SMD:D_SOD-128"
 			(at 49.53 35.56 0)
 			(effects
