File: charging_controller/Hardware/charging_controller.kicad_sch (KiCad schematic)
At the start: 70 parts, among them IC1 VOM1271T, J1 XT30, J10 CAN, J11 HALL2, J12 Pad_TH, J13 B2B, J14 HALL2, J2 XT60, J3 XT30, J4 Conn_01x08_Pin, J7 XT60, Q1 2N7002K, Q3 DMP6023LE-13, SW1 SW_Push, U1 STM32F103CBTx, U2 NCP114BSN330T1G, U3 ACS712xLCTR-20A, U4 MCP2562-E-SN, U5 THN 20WIR

Commit message: last commit before gerber export
Parts:
- renumbered C10 to C1, C8 to C10, C12 to C11, C9 to C12, C14 to C13, C13 to C14, C11 to C2, C7 to C3, C5 to C4, C6 to C5, C1 to C6, C2 to C7, C3 to C8, C4 to C9, D4 to D3, D3 to D4, J2 to J1, J13 to J10, J7 to J2, J1 to J3, J3 to J4, J11 to J5, J14 to J6, J12 to J7, J10 to J8, J4 to J9, Q3 to Q1, Q1 to Q2, R4 to R10, R6 to R11, R5 to R12, R10 to R14, R3 to R2, R11 to R3, R8 to R4, R9 to R5, R7 to R6, R12 to R7, R14 to R8, R2 to R9, TH2 to TH1, U5 to U1, U1 to U3, U3 to U4, U4 to U5

Commit message: shopping list, gerbers and board updates
Parts:
- added IC2: VOM1271T, firo_footprints:SOP254P675X240-4N, symbol VOM1271T:VOM1271T
- added Q3: SIDR392DP-T1-GE3, firo_footprints:PowerPAK_SO-8DC for VISHAY SIDR392DP-T1-GE3, symbol Simulation_SPICE:NMOS
- added R20: 120, Resistor_SMD:R_0805_2012Metric, symbol Device:R
Connections:
- net GND: now also IC2.2 (K_1)
- net at D3.3 (K), U4.1 (IP+), U4.2 (IP+): now also Q3.3 (D); no longer J4.2 (Pin_2)
- net CHG_CUT: now reaches U3.21 (PB10)
- net CHG_CUT: now also R20.1
- new net: IC2.1 (A_1), R20.2
- new net: IC2.3 (K_2), J4.2 (Pin_2), Q3.1 (S)
- new net: IC2.4 (A_2), Q3.2 (G)
Other:
- note removed: "Turn off circuit??"
