File: charging_controller/Hardware/charging_controller.kicad_pcb (KiCad board)
At the start: 4 copper layers, 72.5 x 80 mm, 53 parts, among them J1 XT30, J10 CAN, J2 XT60, J3 XT30, J4 Conn_01x08_Pin, J7 XT60, Q1 2N7002K, Q3 DMP6023LE-13, SW1 SW_Push, U1 STM32F103CBTx, U2 NCP114BSN330T1G, U3 ACS712xLCTR-20A, U4 MCP2562-E-SN, U5 THN 20WIR

Commit message: gaining_a_level_of_exhaustion_xd
Parts:
- removed REF**: PinHeader_2x08_P2.54mm_Vertical, Connector_PinHeader_2.54mm:PinHeader_2x08_P2.54mm_Vertical
- added J11: HALL2, firo_footprints:TEConnectivity_RITS_Header_3P_V, F.Cu at (146.7, 105.7)
- added J12: Pad_TH, firo_footprints:TEConnectivity_RITS_Header_3P_V, F.Cu at (146.7, 119.6)
- added J13: B2B, Connector_PinHeader_2.54mm:PinHeader_2x08_P2.54mm_Vertical, F.Cu at (149.0, 81.4)
- added J14: HALL2, firo_footprints:TEConnectivity_RITS_Header_3P_V, F.Cu at (146.7, 112.2)
- added JP5: Jumper_2_Small_Open, Jumper:SolderJumper-2_P1.3mm_Open_RoundedPad1.0x1.5mm, B.Cu at (152.8, 122.8)
- added R13: R, Resistor_SMD:R_0402_1005Metric, F.Cu at (154.5, 95.8)
- C13, C14, R11, R2, R3, R4, TH2: moved to B.Cu
- moved C7 128.4 mm to (167.6, 91.9)
- moved C10 128.1 mm to (155.1, 112.3)
- moved C14 127.4 mm to (166.2, 110.8), turned to -90 degrees
- moved C13 120.5 mm to (162.7, 105.1)
- moved C9 111.8 mm to (133.6, 125.2)
- moved R4 102.3 mm to (147.4, 114.1)
- moved C11 99.9 mm to (155.1, 106.7)
- moved R6 92.8 mm to (154.6, 96.8)
- moved R5 90.1 mm to (154.8, 101.6), turned to 180 degrees
- moved R2 89.7 mm to (147.4, 107.7)
- moved J10 56.6 mm to (157.5, 120.7), turned to 180 degrees
- moved R10 43.1 mm to (162.6, 114.0), turned to 0 degrees
- moved JP4 42.5 mm to (158.6, 112.9), turned to 90 degrees
- moved JP3 39.6 mm to (168.4, 112.1), turned to -90 degrees
- moved U2 36.6 mm to (155.1, 109.5), turned to 90 degrees
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Connections:
- D1 pad 1: Net-(D1-K) -> +BATT
- J10 pad 1: GND -> Net-(J10-Pin_1)
- Q3 pad 3: Net-(D1-K) -> +BATT
- U1 pad 12: unconnected-(U1-PA2-Pad12) -> A8
- U1 pad 13: unconnected-(U1-PA3-Pad13) -> A5
- U1 pad 14: unconnected-(U1-PA4-Pad14) -> A10
- U1 pad 15: unconnected-(U1-PA5-Pad15) -> CHG_INIT
- U1 pad 16: unconnected-(U1-PA6-Pad16) -> T3
- U1 pad 17: unconnected-(U1-PA7-Pad17) -> T2
- U1 pad 18: unconnected-(U1-PB0-Pad18) -> CHG_CURR
- U1 pad 19: unconnected-(U1-PB1-Pad19) -> T1
- U1 pad 25: unconnected-(U1-PB12-Pad25) -> SENSE
- U1 pad 26: unconnected-(U1-PB13-Pad26) -> HALL1
- U1 pad 27: unconnected-(U1-PB14-Pad27) -> HALL2
- U1 pad 28: unconnected-(U1-PB15-Pad28) -> CANSTBY
- U1 pad 31: unconnected-(U1-PA10-Pad31) -> CANTX
- U1 pad 32: unconnected-(U1-PA11-Pad32) -> CANRX
- U1 pad 43: unconnected-(U1-PB7-Pad43) -> MOT_EN
- U1 pad 45: unconnected-(U1-PB8-Pad45) -> IN2
- U1 pad 46: unconnected-(U1-PB9-Pad46) -> IN1
- U5 pad 3: unconnected-(U5-ROn/Off-Pad3) -> ROn/Off
Routing:
- net SENSE: track 0.00 -> 59.6 mm
- net CHG_CURR: track 0.00 -> 54.1 mm
- net T2: track 0.00 -> 52.1 mm, vias 0 -> 1
- net T1: track 0.00 -> 32.2 mm
- net NRST: track 0.00 -> 32.2 mm, vias 0 -> 1
- net Net-(J2-Pin_2): track 0.00 -> 28.7 mm
- net CHG_INIT: track 0.00 -> 26.8 mm
- net +5V: track 0.00 -> 24.3 mm, vias 0 -> 8
- net HALL2: track 0.00 -> 23.5 mm, vias 0 -> 1
- net IN1: track 0.00 -> 23.5 mm, vias 0 -> 1
- net IN2: track 0.00 -> 22.5 mm, vias 0 -> 1
- net MOT_EN: track 0.00 -> 22.1 mm, vias 0 -> 1
- net HALL1: track 0.00 -> 18.3 mm, vias 0 -> 1
- net A5: track 0.00 -> 15.8 mm
- net CANSTBY: track 0.00 -> 13.4 mm, vias 0 -> 1
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- added copper zone on F.Cu, net +3V3
- added copper zone on F.Cu, net +5V
- added copper zone on B.Cu, net GND
- added copper zone on F.Cu, net Net-(D4-K)
- added copper zone on F.Cu, net Net-(J1-Pin_2)
Other:
- board text added: "CONV"
- board text added: "HALL1"
- board text added: "HALL2"
- board text added: "PAD"
- board text added: "P_THR"

Commit message: PCBs possibly finished + some file org
Parts:
- added D3: G2V4, LED_SMD:LED_0805_2012Metric, F.Cu at (159.4, 77.6)
- added D5: G2V4, LED_SMD:LED_0805_2012Metric, F.Cu at (157.2, 77.6)
- added D6: G2V4, LED_SMD:LED_0805_2012Metric, F.Cu at (155.0, 77.6)
- added D7: B3V1, LED_SMD:LED_0805_2012Metric, F.Cu at (164.6, 77.6)
- added D8: B3V1, LED_SMD:LED_0805_2012Metric, F.Cu at (162.5, 77.6)
- added IC1: VOM1271T, firo_footprints:SOP254P675X240-4N, F.Cu at (142.9, 99.8)
- added R14: 120, Resistor_SMD:R_0402_1005Metric, F.Cu at (143.8, 97.0)
- added R15: 2k2, Resistor_SMD:R_1206_3216Metric, B.Cu at (136.1, 91.7)
- added R16: 240, Resistor_SMD:R_0805_2012Metric, F.Cu at (157.2, 81.0)
- added R17: 120, Resistor_SMD:R_0805_2012Metric, F.Cu at (155.0, 81.0)
- added R18: 20, Resistor_SMD:R_0805_2012Metric, F.Cu at (164.6, 81.0)
- added R19: 20, Resistor_SMD:R_0805_2012Metric, F.Cu at (162.5, 81.0)
- added REF**: FIRO2.1 (h=5mm), firo_ID:FIRO2.1 (h=5mm), F.Cu at (162.6, 65.0)
- added REF**: BLUE_boat_supersmall, BLUE_ID:BLUE_boat_supersmall, B.Cu at (176.0, 77.5)
- D1: value 5V -> 10V
- R1: value ?? -> 47k
- moved Q1 1.02 mm to (136.5, 98.6)
Connections:
- Q1 pad 1: CHG_INIT -> Net-(IC1-A_2)
- U1 pad 4: unconnected-(U1-PC15-Pad4) -> D2
- U1 pad 5: unconnected-(U1-PD0-Pad5) -> D1
Routing:
- net Net-(D3-A): track 0.00 -> 45.4 mm, vias 0 -> 1
- net D1: track 0.00 -> 15.1 mm, vias 0 -> 2
- net D2: track 0.00 -> 14.5 mm, vias 0 -> 2
- net Net-(IC1-A_2): track 0.00 -> 9.73 mm
- net CHG_INIT: track 26.8 -> 19.7 mm
- net Net-(IC1-A_1): track 0.00 -> 5.51 mm
- net Net-(IC1-K_2): track 7.38 -> 11.4 mm
- net +24V: track 13.3 -> 16.6 mm
- net Net-(D7-A): track 0.00 -> 1.56 mm
- net Net-(D8-A): track 0.00 -> 1.56 mm
- net Net-(D6-A): track 0.00 -> 1.55 mm
- net Net-(D5-A): track 0.00 -> 1.55 mm
- net Net-(JP1-A): track 7.44 -> 8.94 mm
- net SENSE: track 59.6 -> 60.7 mm
- net +5V: track 24.3 -> 25.3 mm, vias 8 -> 9
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Other:
- board text added: "#"
- board text added: "+5V"
- board text added: "24V"
- board text added: "3.3V"
- board text added: "3V3"
- board text added: "CAN"
- board text added: "CHG. CONTROL"
- board text added: "FIRO 2.1 ('24) CHARGING CONTROLLER Main board v1, 09.08 PU"
- board text added: "GND"
- board text added: "JNRST"
- board text added: "JP1-NRST SWICH JP2-BOOT0 SEL"
- board text added: "JP3-CAN Vio JP4-CAN SBY"
- board text added: "JTCK"
- board text added: "JTDI"
- board text added: "JTDO"
- board text added: "JTMS"
- board text added: "NRST"
- board text added: "OTH"

Commit message: a lot of work - charging main BOM complete
Parts:
- C4: footprint Capacitor_SMD:C_0402_1005Metric -> Capacitor_SMD:C_0805_2012Metric
- D1: footprint Diode_SMD:D_SOD-123 -> Diode_SMD:D_SOD-128
- D2: footprint Diode_SMD:D_SOD-123 -> Diode_SMD:D_SOD-523
- R1: value 47k -> 39k
- R12: value ?? -> 6k8
- R14: footprint Resistor_SMD:R_0402_1005Metric -> Resistor_SMD:R_0805_2012Metric
- R2, R4: footprint Resistor_SMD:R_0603_1608Metric -> Resistor_SMD:R_0402_1005Metric
- R7: value ?? -> 39k; footprint Resistor_SMD:R_0402_1005Metric -> Resistor_SMD:R_0603_1608Metric
- moved D2 1.01 mm to (143.4, 124.8)
- moved R14 0.70 mm to (144.2, 96.5)
- moved C4 0.68 mm to (167.5, 104.9)
- moved D1 0.49 mm to (125.6, 65.5)
- moved R4 0.39 mm to (147.4, 114.5)
- moved R2 0.22 mm to (147.4, 108.0)
- moved R7 0.13 mm to (123.7, 127.0)
Routing:
- net SENSE: track 60.7 -> 59.7 mm
- net CHG_INIT: track 19.7 -> 18.8 mm
- net +5V: track 25.3 -> 26.1 mm
- net HALL2: track 23.5 -> 24.1 mm

Commit message: last commit before gerber export
Parts:
- R11: renamed from R6; value R -> 5k6
- R12: renamed from R5; value R -> 5k6
- R13: value R -> 5k6
- moved R2 12.2 mm to (116.7, 93.3), turned to 90 degrees
- moved R3 8.78 mm to (118.4, 93.3), turned to -90 degrees
- moved U1 5.06 mm to (125.2, 83.2), turned to 90 degrees
- moved R15 4.37 mm to (132.2, 89.8), turned to 0 degrees
- renumbered C10 to C1, C8 to C10, C12 to C11, C9 to C12, C14 to C13, C13 to C14, C11 to C2, C7 to C3, C5 to C4, C6 to C5, C1 to C6, C2 to C7, C3 to C8, C4 to C9, D4 to D3, D3 to D4, J2 to J1, J13 to J10, J7 to J2, J1 to J3, J3 to J4, J11 to J5, J14 to J6, J12 to J7, J10 to J8, J4 to J9, Q3 to Q1, Q1 to Q2, R4 to R10, R10 to R14, R3 to R2, R11 to R3, R8 to R4, R9 to R5, R7 to R6, R12 to R7, R14 to R8, R2 to R9, TH2 to TH1, U5 to U1, U1 to U3, U3 to U4, U4 to U5
Routing:
- net +24V: track 16.6 -> 51.2 mm
- net Net-(J3-Pin_2): track 6.29 -> 12.3 mm
- net +BATT: track 9.69 -> 12.2 mm
- net Net-(D4-A): track 45.4 -> 46.4 mm
- net GND: vias 273 -> 275
Other:
- board text added: "JP3-CAN Vio JP4-CAN SBY JP5-CAN GND"
- board text removed: "JP3-CAN Vio JP4-CAN SBY"

Commit message: shopping list, gerbers and board updates
Parts:
- added IC2: VOM1271T, firo_footprints:SOP254P675X240-4N, B.Cu at (137.9, 109.5)
- added Q3: SIDR392DP-T1-GE3, firo_footprints:PowerPAK_SO-8DC for VISHAY SIDR392DP-T1-GE3, F.Cu at (132.9, 106.4)
- added R20: 120, Resistor_SMD:R_0805_2012Metric, B.Cu at (136.5, 103.4)
- D3: moved to B.Cu
- moved D3 5.52 mm to (128.7, 106.4), turned to 180 degrees
Connections:
- J4 pad 2: Net-(D3-K) -> Net-(IC2-K_2)
- U3 pad 21: unconnected-(U3-PB10-Pad21) -> CHG_CUT
Routing:
- net CHG_CUT: track 0.00 -> 25.2 mm, vias 0 -> 1
- net Net-(IC2-A_2): track 0.00 -> 13.0 mm, vias 0 -> 1
- net Net-(IC2-K_2): track 0.00 -> 11.0 mm, vias 0 -> 1
- net Net-(IC1-K_2): track 11.4 -> 18.1 mm, vias 0 -> 3
- net Net-(IC2-A_1): track 0.00 -> 2.18 mm
- net Net-(D3-K): vias 0 -> 4
- net GND: vias 275 -> 276
- added copper zone on B.Cu, net Net-(D3-K)
- added copper zone on F.Cu, net Net-(IC2-K_2)
Other:
- board text added: "JLCJLCJLCJLC"

Commit message: port to office
Routing:
- net GND: vias 276 -> 278
Other:
- board text added: "PADTH"
- board text removed: "P_THR"
Changed lines of the file:
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@@
 			(drillshape 0)
 			(scaleselection 1)
-			(outputdirectory "gerber/")
+			(outputdirectory "chh_control_gerber/")
 		)
 	)
@@
 			(end -1.85 1.925)
 			(stroke
-				(width 0.2)
+				(width 0.15)
 				(type solid)
 			)
@@
 			(end 1.85 1.925)
 			(stroke
-				(width 0.2)
+				(width 0.15)
 				(type solid)
 			)
@@
 			(end -1.85 -1.925)
 			(stroke
-				(width 0.2)
+				(width 0.15)
 				(type solid)
 			)
@@
 			(end 1.85 -1.925)
 			(stroke
-				(width 0.2)
+				(width 0.15)
 				(type solid)
 			)
@@
 			(end -2.2 -1.945)
 			(stroke
-				(width 0.2)
+				(width 0.15)
 				(type solid)
 			)
@@
 		(tags "Integrated Circuit")
 		(property "Reference" "IC2"
-			(at 2.4 3.22 90)
+			(at 0 2.8 90)
 			(layer "B.SilkS")
 			(effects
 				(font
-					(size 1.27 1.27)
-					(thickness 0.254)
+					(size 1 1)
+					(thickness 0.15)
 				)
 				(justify mirror)
@@
 			(end -3.95 1.945)
 			(stroke
-				(width 0.2)
+				(width 0.15)
 				(type solid)
 			)
@@
 			(end -1.85 -1.925)
 			(stroke
-				(width 0.2)
+				(width 0.15)
 				(type solid)
 			)
@@
 			(end -1.85 1.925)
 			(stroke
-				(width 0.2)
+				(width 0.15)
 				(type solid)
 			)
@@
 			(end 1.85 -1.925)
 			(stroke
-				(width 0.2)
+				(width 0.15)
 				(type solid)
 			)
@@
 			(end 1.85 1.925)
 			(stroke
-				(width 0.2)
+				(width 0.15)
 				(type solid)
 			)
@@
 	)
 	(gr_text "HALL2"
-		(at 136.6 108.8 -90)
+		(at 136.453589 108.869012 270)
 		(layer "F.SilkS" knockout)
 		(effects
 			(font
-				(size 1.5 1.5)
+				(size 1.5 1.4)
 				(thickness 0.3)
 				(bold yes)
@@
 		)
 	)
-	(gr_text "P_THR"
-		(at 136.8 116.1 270)
+	(gr_text "PADTH"
+		(at 136.5 116.1 270)
 		(layer "F.SilkS" knockout)
 		(effects
 			(font
-				(size 1.4 1.44)
+				(size 1.5 1.44)
 				(thickness 0.3)
 				(bold yes)
@@
 	)
 	(gr_text "HALL1"
-		(at 136.6 102.1 -90)
+		(at 136.45366 102.368834 270)
 		(layer "F.SilkS" knockout)
 		(effects
 			(font
-				(size 1.5 1.5)
+				(size 1.5 1.4)
 				(thickness 0.3)
 				(bold yes)
@@
 	)
 	(via
+		(at 139.2 104.9)
+		(size 0.45)
+		(drill 0.2)
+		(layers "F.Cu" "B.Cu")
+		(free yes)
+		(net 2)
+	)
+	(via
 		(at 166.087488 61.281377)
 		(size 0.45)
@@
 	)
 	(via
+		(at 139.2 108.2)
+		(size 0.45)
+		(drill 0.2)
+		(layers "F.Cu" "B.Cu")
+		(free yes)
+		(net 2)
+	)
+	(via
 		(at 155.707 113.284)
 		(size 0.45)
@@
 	)
 	(via
-		(at 137.5 102.5)
+		(at 138.2 102.1)
 		(size 0.45)
 		(drill 0.2)
@@
 	)
 	(via
-		(at 137.5 105)
+		(at 137.4 108.7)
 		(size 0.45)
 		(drill 0.2)
