File: pad_motor_controller/Hardware/pad_motor_controller.kicad_sch (KiCad schematic)
At the start: 19 parts, among them J1 ??, J2 Conn_01x02_MountingPin, J3 B2B, Q1 DMP6023LE-13, U1 L6201PS

Commit message: PCBs possibly finished + some file org
Parts:
- removed D1, D2: DST5100S-A, Package_TO_SOT_SMD:TO-277B, symbol Device:D_Schottky
- removed H3, H4: MountingHole_Pad, MountingHole:MountingHole_3.2mm_M3_Pad_Via, symbol Mechanical:MountingHole_Pad
- added D1, D2: DST5100S, Package_TO_SOT_SMD:TO-277B, symbol Device:D_Schottky_AAK
- added D4: G2V4, LED_SMD:LED_0805_2012Metric, symbol Device:LED
- added R3: 3k9, Resistor_SMD:R_1206_3216Metric, symbol Device:R
- J1: footprint (none) -> firo_footprints:WAGO 2601-3102
- Q1: footprint Package_TO_SOT_SMD:TO-252-2 -> Package_TO_SOT_SMD:SOT-223-3_TabPin2
Connections:
- net +BATT: now also R3.1
- net GND: now also U1.21 (GND), D1.1 (A), D1.2 (A), D2.1 (A), D2.2 (A), D4.1 (K)
- net at C3.1, J1.2 (Pin_2), R1.2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: now also D2.3 (K)
- net at C2.2, C4.1, J1.1 (Pin_1)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: now also D1.3 (K)
- net at U1.15 (Vref): now also J3.8 (Pin_8); no longer J3.10 (Pin_10)
- net at U1.16 (SENSE): now also J3.10 (Pin_10); no longer J3.8 (Pin_8)
- new net: D4.2 (A), R3.2

Commit message: last commit before gerber export
Parts:
- added JP1: Jumper_2_Small_Open, Jumper:SolderJumper-2_P1.3mm_Open_RoundedPad1.0x1.5mm, symbol Jumper:Jumper_2_Small_Open
- added JP2: Jumper_2_Small_Bridged, Jumper:SolderJumper-2_P1.3mm_Bridged2Bar_RoundedPad1.0x1.5mm, symbol Jumper:Jumper_2_Small_Bridged
- added R2: Current sense (opt), Resistor_SMD:R_1206_3216Metric, symbol Device:R_Small
- C4: value ?? -> 27nF; footprint Capacitor_SMD:C_1206_3216Metric -> Capacitor_SMD:C_0805_2012Metric
- D1: renamed from D3; value 5V -> 10V
- R1: renamed from R2; value ?? -> 39k; footprint Resistor_SMD:R_0805_2012Metric -> Resistor_SMD:R_0603_1608Metric
- R3: renamed from R1; value ?? -> 10
- renumbered D1 to D2, D2 to D3, J2 to J1, J3 to J2, J1 to J3, R3 to R4
Connections:
- net GND: now also JP2.1 (A), R2.1
- net at U1.16 (SENSE): now also JP1.2 (B), JP2.2 (B), R2.2; no longer J2.10 (Pin_10)
- new net: J2.10 (Pin_10), JP1.1 (A)
