File: pad_motor_controller/Hardware/pad_motor_controller.kicad_pcb (KiCad board)
At the start: 2 copper layers, 0 parts

Commit message: PCBs possibly finished + some file org
Parts:
- added C1: 100nF, Capacitor_SMD:C_0805_2012Metric, B.Cu at (206.5, 96.9)
- added C2: 10nF, Capacitor_SMD:C_0805_2012Metric, F.Cu at (211.5, 94.0)
- added C3: 10nF, Capacitor_SMD:C_0805_2012Metric, F.Cu at (211.1, 101.9)
- added C4: ??, Capacitor_SMD:C_1206_3216Metric, F.Cu at (213.2, 108.2)
- added D1: DST5100S, Package_TO_SOT_SMD:TO-277B, F.Cu at (192.2, 124.7)
- added D2: DST5100S, Package_TO_SOT_SMD:TO-277B, F.Cu at (192.2, 108.1)
- added D3: 5V, Diode_SMD:D_SOD-123, B.Cu at (208.7, 86.9)
- added D4: G2V4, LED_SMD:LED_0805_2012Metric, F.Cu at (212.9, 90.6)
- added H1: MountingHole_Pad, MountingHole:MountingHole_3.2mm_M3_Pad_Via, F.Cu at (209.9, 71.7)
- added H2: MountingHole_Pad, MountingHole:MountingHole_3.2mm_M3_Pad_Via, F.Cu at (209.9, 116.7)
- added J1: ??, firo_footprints:WAGO 2601-3102, F.Cu at (200.4, 117.9)
- added J2: Conn_01x02_MountingPin, Connector_AMASS:AMASS_XT60PW-M_1x02_P7.20mm_Horizontal, F.Cu at (193.5, 82.3)
- added J3: B2B, Connector_PinHeader_2.54mm:PinHeader_2x08_P2.54mm_Vertical, F.Cu at (182.9, 87.1)
- added Q1: DMP6023LE-13, Package_TO_SOT_SMD:SOT-223-3_TabPin2, B.Cu at (209.3, 80.9)
- added R1: ??, Resistor_SMD:R_1206_3216Metric, F.Cu at (208.3, 108.2)
- added R2: ??, Resistor_SMD:R_0805_2012Metric, B.Cu at (214.0, 83.2)
- added R3: 3k9, Resistor_SMD:R_1206_3216Metric, B.Cu at (211.5, 90.2)
- added REF**: F2_med, firo_ID:F2_med, F.Cu at (210.4, 81.4)
- added REF**: BLUE_boat_supersmall, BLUE_ID:BLUE_boat_supersmall, B.Cu at (201.0, 108.5)
- added TH1: Board_TH, Resistor_SMD:R_0603_1608Metric, F.Cu at (197.9, 106.2)
- added U1: L6201PS, Package_SO:HSOP-20-1EP_11.0x15.9mm_P1.27mm_SlugDown, F.Cu at (200.7, 96.3)
Routing:
- net Net-(D1-K): track 0.00 -> 53.0 mm
- net Net-(D2-K): track 0.00 -> 36.5 mm
- net Net-(J3-Pin_2): track 0.00 -> 27.2 mm, vias 0 -> 1
- net Net-(J2-Pin_1): track 0.00 -> 24.0 mm
- net Net-(U1-BOOT2): track 0.00 -> 22.8 mm, vias 0 -> 12
- net Net-(J3-Pin_12): track 0.00 -> 14.3 mm
- net +BATT: track 0.00 -> 14.0 mm, vias 0 -> 6
- net Net-(J3-Pin_6): track 0.00 -> 12.4 mm
- net Net-(J3-Pin_4): track 0.00 -> 9.81 mm
- net Net-(J3-Pin_8): track 0.00 -> 9.28 mm, vias 0 -> 1
- net Net-(J3-Pin_10): track 0.00 -> 8.55 mm, vias 0 -> 1
- net Net-(D3-A): track 0.00 -> 5.73 mm
- net Net-(U1-BOOT1): track 0.00 -> 3.21 mm
- net Net-(D4-A): track 0.00 -> 2.42 mm, vias 0 -> 1
- net Net-(C4-Pad2): track 0.00 -> 1.89 mm
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- added copper zone on B.Cu, net +BATT
- added copper zone on F.Cu, net +BATT
- added copper zone on B.Cu, net GND
- added copper zone on F.Cu, net GND
- added copper zone on In1.Cu, net GND
- added copper zone on In2.Cu, net GND
- added copper zone on B.Cu, net Net-(U1-BOOT2)
- added copper zone on F.Cu, net Net-(U1-BOOT2)
Other:
- board outline added: 35.6 x 65 mm
- copper layers 2 -> 4
- board text added: "#"
- board text added: "FIRO 2.1 ('24) CHARGING CONTROLLER Motor v1, 09.08 PU"
- board text added: "VBAT"

Commit message: last commit before gerber export
Parts:
- added JP1: Jumper_2_Small_Open, Jumper:SolderJumper-2_P1.3mm_Open_RoundedPad1.0x1.5mm, B.Cu at (133.9, 97.7)
- added JP2: Jumper_2_Small_Bridged, Jumper:SolderJumper-2_P1.3mm_Bridged2Bar_RoundedPad1.0x1.5mm, B.Cu at (137.2, 100.4)
- added R4: Current sense (opt), Resistor_SMD:R_1206_3216Metric, B.Cu at (134.8, 101.2)
- C4: footprint Capacitor_SMD:C_1206_3216Metric -> Capacitor_SMD:C_0805_2012Metric
- D3: value 5V -> 10V
- R1: value ?? -> 10
- R2: value ?? -> 39k; footprint Resistor_SMD:R_0805_2012Metric -> Resistor_SMD:R_0603_1608Metric
- moved R2 54.9 mm to (159.1, 84.2)
- moved C4 54.8 mm to (158.4, 108.6)
- moved C3 54.7 mm to (156.4, 102.2)
- moved D2 54.7 mm to (137.5, 108.5)
- moved Q1 54.7 mm to (154.6, 81.3)
- moved R3 54.7 mm to (156.8, 90.6)
- moved TH1 54.7 mm to (143.2, 106.6)
- moved C1 54.7 mm to (151.9, 97.3)
- moved C2 54.7 mm to (156.8, 94.4)
- moved D1 54.7 mm to (137.5, 125.1)
- moved D3 54.7 mm to (154.0, 87.3)
- moved D4 54.7 mm to (158.2, 91.0)
- moved H1 54.7 mm to (155.2, 72.1)
- moved H2 54.7 mm to (155.2, 117.1)
- moved J1 54.7 mm to (145.7, 118.3)
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Connections:
- U1 pad 16: Net-(J3-Pin_10) -> Net-(JP1-B)
Routing:
- net Net-(JP1-B): track 0.00 -> 6.36 mm, vias 0 -> 8
- net Net-(J3-Pin_10): track 8.55 -> 2.40 mm, vias 1 -> 0
- net Net-(J3-Pin_6): track 12.4 -> 13.2 mm
- net Net-(J3-Pin_8): track 9.28 -> 8.76 mm
- net +BATT: vias 6 -> 8
- net GND: vias 273 -> 276
- added copper zone on B.Cu, net Net-(JP1-B)
- added copper zone on F.Cu, net Net-(JP1-B)
Other:
- board text added: "JP2 MUST BE SOLDERED IN ADD. TO COPPER"
- board text added: "UNLESS R4 USED"

Commit message: shopping list, gerbers and board updates
Other:
- board text added: "JLCJLCJLCJLC"
Changed lines of the file:
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@@
 			(plot_on_all_layers_selection 0x0000000_00000000)
 			(disableapertmacros no)
-			(usegerberextensions no)
-			(usegerberattributes yes)
-			(usegerberadvancedattributes yes)
-			(creategerberjobfile yes)
+			(usegerberextensions yes)
+			(usegerberattributes no)
+			(usegerberadvancedattributes no)
+			(creategerberjobfile no)
 			(dashed_line_dash_ratio 12.000000)
 			(dashed_line_gap_ratio 3.000000)
@@
 			(psa4output no)
 			(plotreference yes)
-			(plotvalue yes)
+			(plotvalue no)
 			(plotfptext yes)
 			(plotinvisibletext no)
 			(sketchpadsonfab no)
-			(subtractmaskfromsilk no)
+			(subtractmaskfromsilk yes)
 			(outputformat 1)
 			(mirror no)
-			(drillshape 1)
+			(drillshape 0)
 			(scaleselection 1)
-			(outputdirectory "")
+			(outputdirectory "pad_motor_gerber/")
 		)
 	)
@@
 		)
 	)
+	(gr_text "JLCJLCJLCJLC"
+		(at 137.2 71.1 0)
+		(layer "F.SilkS")
+		(effects
+			(font
+				(size 1 1)
+				(thickness 0.15)
+			)
+			(justify left bottom)
+		)
+	)
