File: temp_power_management/Hardware/temp_power_management.kicad_pcb (KiCad board)
At the start: 2 copper layers, 71 parts, among them J1 BAT1_IN, J10 BAT_OUT6, J11 USB_A_Stacked, J12 USB_A_Stacked, J13 PC_Conv_CTRL, J14 CAN, J15 Conn_01x08_Pin, J2 BAT2_IN, J3 CHG_PORT, J4 5V_Conv_Conn, J5 BAT_OUT1, J6 BAT_OUT2, J7 BAT_OUT3, J8 BAT_OUT4, J9 BAT_OUT5, K1 RELPOL R40N, Q1 SUM110P06-07L-E3, Q2 SUM110P06-07L-E3, Q3 2N7002K, SW1 EMERG_nSTOP, SW2 EMERG_nSTOP, SW3 EMERG_STOP, SW4 SW_Push, U1 NCP114BSN330T1G, U2 STM32F103CBTx, U3 MCP2562-E-SN

Commit message: temp_pms bloody FINISHED and ordered.
Parts:
- removed C6: 100nF, Capacitor_SMD:C_0402_1005Metric
- added D10: G2V4, LED_SMD:LED_0805_2012Metric, F.Cu at (117.3, 94.7)
- added D11: G2V4, LED_SMD:LED_0805_2012Metric, F.Cu at (119.9, 94.7)
- added D8: B3V1, LED_SMD:LED_0805_2012Metric, F.Cu at (121.9, 64.8)
- added D9: B3V1, LED_SMD:LED_0805_2012Metric, F.Cu at (119.6, 64.8)
- added FB1: FerriteBead_Small, Resistor_SMD:R_0402_1005Metric_Pad0.72x0.64mm_HandSolder, B.Cu at (117.2, 67.8)
- added H1: MountingHole_Pad, MountingHole:MountingHole_3.2mm_M3_Pad_Via, F.Cu at (195.1, 73.2)
- added R19: 20, Resistor_SMD:R_0805_2012Metric, B.Cu at (121.9, 66.7)
- added R20: 20, Resistor_SMD:R_0805_2012Metric, B.Cu at (119.6, 66.7)
- added R21: 240, Resistor_SMD:R_0805_2012Metric, F.Cu at (117.3, 91.3)
- added R22: 120, Resistor_SMD:R_0805_2012Metric, F.Cu at (119.9, 91.3)
- added R23: 10k, Resistor_SMD:R_0402_1005Metric, B.Cu at (105.4, 89.2)
- added R24: 10k, Resistor_SMD:R_0402_1005Metric, B.Cu at (105.4, 88.1)
- added R25: 10k, Resistor_SMD:R_0402_1005Metric, B.Cu at (121.9, 70.6)
- added R26: 10k, Resistor_SMD:R_0402_1005Metric, B.Cu at (121.9, 71.6)
- added R27: R, Resistor_SMD:R_0402_1005Metric, B.Cu at (181.1, 74.4)
- added REF**: FIRO2.1 (h=5mm), firo_ID:FIRO2.1 (h=5mm), F.Cu at (130.6, 91.5)
- added REF**: BLUE_boat_supersmall, BLUE_ID:BLUE_boat_supersmall, B.Cu at (181.4, 122.9)
- C1, C11, C12, C2, C3, C4, C5, C7, C8, C9, D1, D3, D6, D7, JP1, JP3, JP4, JP5, Q1, Q2, Q3, R1, R10, R11, R14, R15, R16, R17, R18, R2, R3, R4, R5, R6, R8, R9, RV1, U1, U2, U3: moved to B.Cu
- moved C9 147.1 mm to (116.7, 69.3), turned to 180 degrees
- moved C10 145.0 mm to (112.3, 60.7), turned to -90 degrees
- moved R5 142.7 mm to (194.1, 66.8), turned to 0 degrees
- moved Q3 142.6 mm to (193.5, 64.3), turned to 90 degrees
- moved R4 140.1 mm to (194.1, 67.8), turned to 180 degrees
- moved D2 139.0 mm to (190.2, 64.3), turned to -90 degrees
- moved C7 133.5 mm to (110.5, 71.9), turned to 180 degrees
- moved R7 133.4 mm to (190.2, 68.3), turned to -90 degrees
- moved C8 132.3 mm to (113.2, 83.1)
- moved C4 132.0 mm to (121.7, 78.2), turned to 90 degrees
- moved C3 130.2 mm to (112.3, 69.8), turned to 180 degrees
- moved SW4 129.4 mm to (115.6, 60.5), turned to 180 degrees
- moved U2 128.5 mm to (115.6, 75.7), turned to -90 degrees
- moved D5 127.5 mm to (186.4, 64.3), turned to -90 degrees
- moved C5 125.0 mm to (113.0, 81.5)
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Connections:
- C9 pad 1: +3V3 -> Net-(U2-VDDA)
- J13 pad MP: (no net) -> GND
- U2 pad 12: unconnected-(U2-PA2-Pad12) -> D1
- U2 pad 13: unconnected-(U2-PA3-Pad13) -> D2
- U2 pad 14: unconnected-(U2-PA4-Pad14) -> RC
- U2 pad 17: unconnected-(U2-PA7-Pad17) -> T2
- U2 pad 18: unconnected-(U2-PB0-Pad18) -> BUS_VOLTAGE
- U2 pad 19: unconnected-(U2-PB1-Pad19) -> 5V_VOLTAGE
- U2 pad 33: unconnected-(U2-PA12-Pad33) -> CANSTBY
- U2 pad 42: unconnected-(U2-PB6-Pad42) -> PC_REMOTE
- U2 pad 9: +3V3 -> Net-(U2-VDDA)
Routing:
- net RC: track 0.00 -> 77.0 mm
- net T2: track 0.00 -> 76.6 mm, vias 0 -> 1
- net Off42V: track 0.00 -> 70.9 mm, vias 0 -> 1
- net +VDC: track 0.00 -> 70.8 mm
- net +BATT: track 0.00 -> 68.6 mm, vias 0 -> 1
- net BUS_VOLTAGE: track 0.00 -> 59.1 mm
- net OnGND: track 0.00 -> 58.5 mm
- net 5V_VOLTAGE: track 0.00 -> 39.6 mm
- net On42V: track 0.00 -> 38.7 mm
- net NRST: track 0.00 -> 31.4 mm, vias 0 -> 1
- net +3V3: track 0.00 -> 22.8 mm, vias 0 -> 13
- net PC_REMOTE: track 0.00 -> 22.3 mm, vias 0 -> 1
- net JTDO/TRACESWO: track 0.00 -> 22.2 mm
- net CANRX: track 0.00 -> 22.0 mm
- net JTCK/SWCLK: track 0.00 -> 21.1 mm
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- added copper zone on In1.Cu, net +3V3
- added copper zone on B.Cu, net +5V
- added copper zone on F.Cu, net +5V
- added copper zone on In1.Cu, net +5V
- added copper zone on B.Cu, net +BATT
- added copper zone on B.Cu, net +VDC
- added copper zone on F.Cu, net +VDC
- added copper zone on B.Cu, net /SFT_IM
- added copper zone on B.Cu, net GND
- added copper zone on F.Cu, net GND
- added copper zone on In1.Cu, net GND
- added copper zone on In2.Cu, net GND
- added copper zone on B.Cu, net Net-(J1-Pin_2)
- added copper zone on F.Cu, net Net-(J1-Pin_2)
- added copper zone on In1.Cu, net Net-(J1-Pin_2)
- added copper zone on In2.Cu, net Net-(J1-Pin_2)
- added copper zone on B.Cu, net Net-(J1-Pin_3)
- added copper zone on F.Cu, net Net-(J1-Pin_3)
- added copper zone on B.Cu, net Net-(Q1-D)
Other:
- board outline added: 100 x 85 mm
- copper layers 2 -> 4
- board text added: "#"
- board text added: "+5V"
- board text added: "11"
- board text added: "12"
- board text added: "21"
- board text added: "22"
- board text added: "28-42VDC"
- board text added: "33"
- board text added: "34"
- board text added: "3V3"
- board text added: "5V OUTPUT"
- board text added: "BAT1"
- board text added: "BAT2"
- board text added: "BATTERY VOLTAGE OUTPUT"
- board text added: "CAN"
- board text added: "CHARGING"
- board text added: "D1"
- board text added: "D2"
- board text added: "DO NOT OPERATE WHEN FAULT LIT"
- board text added: "EMERGENCY SWITCH CONNECTION"
- board text added: "FAULT"
- board text added: "FIRO 2.1 ('24) POWER MANAGEMENT BOARD TEMPORARY v1, 023.08 PU"
- board text added: "GND"
- board text added: "JLCJLCJLCJLC"
- board text added: "JNRST"
- board text added: "JTCK"
- board text added: "JTDI"
- board text added: "JTDO"
- board text added: "JTMS"
- board text added: "NRST"
- board text added: "PC SUPPLY CONTROL"
- board text added: "POWER MGMT BOARD"
- board text added: "PROGRAMMING"
- board text added: "TO NORMALLY CLOSED"
- board text added: "TO NORMALLY OPEN"
- board text added: "VBAT"
- board text added: "VDC"
