File: temp_power_management/Hardware/temp_power_management.kicad_sch (KiCad schematic)
At the start: 34 parts, among them J1 BAT1_IN, J10 CAN, J11 Conn_01x08_Pin, J2 BAT_OUT1, J3 BAT2_IN, J4 BAT_OUT2, J5 BAT_OUT3, J6 BAT_OUT4, J7 BAT_OUT5, J8 BAT_OUT5, J9 CHG_PORT, K1 RELPOL R40N-3021-85-1024, Q1 SIDR392DP-T1-GE3, SW1 SW_Push, SW2 SW_Push_Open, U1 STM32F103CBTx, U2 NCP114BSN330T1G

Commit message: minor work, updates to shopping list
Parts:
- added D3, D4: LED, symbol Device:LED
- added R10, R4, R5, R6, R9: R, symbol Device:R
- SW2: value SW_Push_Open -> EMERG_STOP
Connections:
- net +BATT: now also SW2.1 (A), R9.2
- net +VDC: now also R10.2
- net -BATT: now also K1.A1, R3.1, D3.1 (K), R6.2
- net GND: now also D4.1 (K)
- net at C11.1, K1.A2: now also R4.2
- net nSTOP: now reaches SW2.2 (B)
- net nSTOP: now also R4.1, R5.1
- net at Q1.2 (G): now also R5.2, R6.1
- new net: D3.2 (A), R9.1
- new net: D4.2 (A), R10.1
Other:
- moved on the sheet: C11, J1, J2, J3, J4, J5, J6, J7, J8, J9, K1, Q1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

Commit message: minor work done
Parts:
- added J12: 5V Converter IN, symbol Connector_Generic:Conn_01x07
- added J13: 5V Converter OUT, symbol Connector_Generic:Conn_01x06
Connections:
- net +5V: now also J13.3 (Pin_3), J13.4 (Pin_4), J13.5 (Pin_5), J13.6 (Pin_6)
- net +VDC: now also J12.4 (Pin_4), J12.5 (Pin_5)
- net GND: now also J12.6 (Pin_6), J12.7 (Pin_7), J13.1 (Pin_1), J13.2 (Pin_2)
- new net RC: J12.1 (Pin_1)
- new net TR: J12.2 (Pin_2)

Commit message: temp_PMS - much done, kill me
Parts:
- removed J12: 5V Converter IN, symbol Connector_Generic:Conn_01x07
- removed J13: 5V Converter OUT, symbol Connector_Generic:Conn_01x06
- removed Q1: SIDR392DP-T1-GE3, firo_footprints:PowerPAK_SO-8DC for VISHAY SIDR392DP-T1-GE3, symbol Simulation_SPICE:NMOS
- added C12, C13: 100nF, Capacitor_SMD:C_0402_1005Metric, symbol Device:C_Small
- added D1, D2: LED, symbol Device:LED
- added D5: D_Schottky, symbol Device:D_Schottky
- added D6: D_Zener, symbol Device:D_Zener
- added F1: 20A?, symbol Device:Fuse_Small
- added J12, J13: USB_A_Stacked, Connector_USB:USB_A_CUI_UJ2-ADH-TH_Horizontal_Stacked, symbol Connector:USB_A_Stacked
- added J14: 5V_Conv_Conn, firo_footprints:MeanWell NID100-R3, symbol Connector_Generic:Conn_01x13
- added JP4, JP5: SolderJumper_3_Bridged12, Jumper:SolderJumper-3_P1.3mm_Bridged12_RoundedPad1.0x1.5mm, symbol Jumper:SolderJumper_3_Bridged12
- added Q3: 2N7002K, Package_TO_SOT_SMD:SOT-23, symbol Transistor_FET:2N7002K
- added Q4: NTR5105PT1G, Package_TO_SOT_SMD:SOT-223-3_TabPin2, symbol Device:Q_PMOS_GDS
- added Q5, Q6: SIDR392DP-T1-GE3, firo_footprints:PowerPAK_SO-8DC for VISHAY SIDR392DP-T1-GE3, symbol Simulation_SPICE:NMOS
- added R11, R12, R14, R15, R16, R17, R18, R19, R20, R21: R, symbol Device:R
- added R7: 120, Resistor_SMD:R_0805_2012Metric, symbol Device:R_Small
- added R8: 5k6, Resistor_SMD:R_0402_1005Metric, symbol Device:R
- added SW3: EMERG_STOP, Button_Switch_SMD:SW_SPST_EVQP7C, symbol Switch:SW_Push
- added TH1: Board_TH, Resistor_SMD:R_0603_1608Metric, symbol Device:Thermistor
- added U3: MCP2562-E-SN, Package_SO:SOIC-8_3.9x4.9mm_P1.27mm, symbol Interface_CAN_LIN:MCP2562-E-SN
- K1: value RELPOL R40N-3021-85-1024 -> RELPOL R40N
- SW2: value EMERG_STOP -> EMERG_nSTOP
Connections:
- net +3V3: now also JP4.1 (A), R8.1
- net +5V: now also C13.2, J12.1 (VBUS1), J12.5 (VBUS2), J13.1 (VBUS1), J13.5 (VBUS2), J14.1 (Pin_1), J14.2 (Pin_2), J14.3 (Pin_3), J14.4 (Pin_4), JP4.3 (B), U3.3 (VDD)
- net +BATT: now also F1.1, Q4.3 (S), R14.2, R18.2, SW3.1; no longer K1.11
- net +VDC: now also D5.1 (K), J14.10 (Pin_10), J14.9 (Pin_9), Q6.3 (D), R11.2, R15.2
- net -BATT: now also R6.1, D2.1 (K), Q3.2 (S), Q5.1 (S), R16.1, R21.1; no longer R6.2
- net CAN+: now also R7.1, U3.7 (CANH)
- net CAN-: now also R7.2, U3.6 (CANL)
- net GND: now also C12.1, C13.1, D5.2 (A), D6.2 (A), J12.4 (GND1), J12.8 (GND2), J12.9 (Shield), J13.4 (GND1), J13.8 (GND2), J13.9 (Shield), J14.5 (Pin_5), J14.6 (Pin_6), J14.7 (Pin_7), J14.8 (Pin_8), JP5.1 (A), Q5.3 (D), Q6.1 (S), R12.1, R19.1, TH1.2, U3.2 (VSS)
- net RC: now also J14.13 (Pin_13)
- net TR: now also J14.12 (Pin_12)
- net On42V: now reaches R5.2
- net On42V: now also R4.1, SW2.2 (B); no longer R6.1
- net CANTX: now reaches U1.31 (PA10)
- net CANTX: now also U3.1 (TXD)
- net CANRX: now reaches U1.32 (PA11)
- net CANRX: now also U3.4 (RXD)
- removed net nSTOP: R4.1, R5.1, SW2.2 (B)
- new net: C12.2, JP4.2 (C), U3.5 (Vio)
- new net: D2.2 (A), R17.1
- new net: Q3.1 (G), R15.1, R16.2
- new net: Q6.2 (G), R20.1, R21.2
- new net: Q4.1 (G), R18.1, R19.2
- new net: D1.1 (K), Q3.3 (D)
- new net: D1.2 (A), R14.1
- new net: JP5.2 (C), U3.8 (STBY)
- new net: Q5.2 (G), R5.1, R6.2
- new net: F1.2, K1.11
- new net: Q4.2 (D), R17.2
- new net BUS_VOLTAGE: D6.1 (K), R11.1, R12.2
- new net CANSTBY: JP5.3 (B)
- new net Off42V: R20.2, SW3.2
- new net T2: R8.2, TH1.1
- no-connect marks 1 -> 10
Other:
- moved on the sheet: C1, C10, C11, C2, C3, C4, C5, C6, C7, C8, C9, D3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

Commit message: port to office
Other:
- note added: "tutaj dioda idealna!!!"
Changed lines of the file:
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@@
+		)
+	)
+	(text "tutaj dioda idealna!!!"
+		(exclude_from_sim no)
+		(at 80.01 49.53 0)
+		(effects
+			(font
+				(size 1.27 1.27)
+				(color 255 121 83 1)
+			)
 		)
 	)

Commit message: power management progress
Parts:
- removed C11: 47uF, Capacitor_SMD:C_2220_5750Metric, symbol Device:C
- removed D2: LED, symbol Device:LED
- removed D5: D_Schottky, symbol Device:D_Schottky
- removed Q4: NTR5105PT1G, Package_TO_SOT_SMD:SOT-223-3_TabPin2, symbol Device:Q_PMOS_GDS
- removed Q5, Q6: SIDR392DP-T1-GE3, firo_footprints:PowerPAK_SO-8DC for VISHAY SIDR392DP-T1-GE3, symbol Simulation_SPICE:NMOS
- removed R17, R18, R19, R20, R21, R5, R6: R, symbol Device:R
- removed R3: 240, Resistor_SMD:R_0805_2012Metric, symbol Device:R_Small
- added D1: 10V, Diode_SMD:D_SOD-128, symbol Device:D_Zener
- added D3: 824520331, Diode_SMD:D_SOD-128, symbol Device:D_Zener
- added D6: D_Zener, Diode_SMD:D_SOD-523, symbol Device:D_Zener
- added J13: PC_Conv_CTRL, firo_footprints:TEConnectivity_RITS_Header_3P_V, symbol Connector_Generic:Conn_01x03
- added Q1, Q2: SUM110P06-07L-E3, Package_TO_SOT_SMD:TO-263-2, symbol Device:Q_PMOS_GDS
- added R1, R15, R16: R, Resistor_SMD:R_0402_1005Metric, symbol Device:R
- added R11: TRIM_R, Resistor_SMD:R_0805_2012Metric, symbol Device:R_Small
- added R2, R3: R, Resistor_SMD:R_0805_2012Metric, symbol Device:R
- added RV1: AV30K1812801NIR1HT, Resistor_SMD:R_1812_4532Metric, symbol Device:Varistor
- added SW2: EMERG_nSTOP, firo_footprints:WAGO 2601-3102, symbol Switch:SW_Push_Open
- D2: renamed from D1; footprint (none) -> LED_SMD:LED_0805_2012Metric
- D4: renamed from D3; footprint (none) -> LED_SMD:LED_0805_2012Metric
- D5: renamed from D4; footprint (none) -> LED_SMD:LED_0805_2012Metric
- D7: renamed from D6; footprint (none) -> Diode_SMD:D_SOD-523
- F1: footprint (none) -> firo_footprints:firo_fuse
- J1: footprint (none) -> firo_footprints:AMASS_MR60-M_1x03_Vertical
- J10: renamed from J8; value BAT_OUT5 -> BAT_OUT6; footprint (none) -> Connector_AMASS:AMASS_XT60-F_1x02_P7.20mm_Vertical
- J2: renamed from J3; footprint (none) -> firo_footprints:AMASS_MR60-M_1x03_Vertical
- J3: renamed from J9; footprint (none) -> Connector_AMASS:AMASS_XT30U-M_1x02_P5.0mm_Vertical
- J5: renamed from J2; footprint (none) -> Connector_AMASS:AMASS_XT60-F_1x02_P7.20mm_Vertical
- J6: renamed from J4; footprint (none) -> Connector_AMASS:AMASS_XT60-F_1x02_P7.20mm_Vertical
- J7: renamed from J5; footprint (none) -> Connector_AMASS:AMASS_XT60-F_1x02_P7.20mm_Vertical
- J8: renamed from J6; footprint (none) -> Connector_AMASS:AMASS_XT60-F_1x02_P7.20mm_Vertical
- J9: renamed from J7; footprint (none) -> Connector_AMASS:AMASS_XT60-F_1x02_P7.20mm_Vertical
- R12: renamed from R9; footprint (none) -> Resistor_SMD:R_1206_3216Metric
- R13: renamed from R10; footprint (none) -> Resistor_SMD:R_1206_3216Metric
- R17: renamed from R11; footprint (none) -> Resistor_SMD:R_0402_1005Metric
- R18: renamed from R12; footprint (none) -> Resistor_SMD:R_0402_1005Metric
- R4: renamed from R15; footprint (none) -> Resistor_SMD:R_0402_1005Metric
- R5: renamed from R16; footprint (none) -> Resistor_SMD:R_0402_1005Metric
- R6: renamed from R4; footprint (none) -> Resistor_SMD:R_1206_3216Metric
- R7: renamed from R14; footprint (none) -> Resistor_SMD:R_1206_3216Metric
- SW1: renamed from SW2; footprint (none) -> firo_footprints:WAGO 2601-3102
- SW3: footprint Button_Switch_SMD:SW_SPST_EVQP7C -> firo_footprints:WAGO 2601-3102
- renumbered C2 to C1, C1 to C10, C12 to C11, C13 to C12, C3 to C2, C4 to C3, C5 to C4, C6 to C5, C7 to C6, C8 to C7, C9 to C8, C10 to C9, J12 to J11, J13 to J12, J10 to J14, J11 to J15, J14 to J4, JP4 to JP3, JP5 to JP4, JP3 to JP5, R7 to R10, R8 to R14, R1 to R8, R2 to R9, SW1 to SW4, U2 to U1, U1 to U2
Connections:
- net -BATT is gone; now on net GND: D4.1 (K), J1.1 (Pin_1), J2.1 (Pin_1), J3.1 (Pin_1), K1.A1, Q3.2 (S), R5.1
- net +5V: now also R15.2
- net +BATT: now also D1.1 (K), Q1.3 (S), Q2.3 (S), R2.1; no longer F1.1, J1.3 (Pin_3), J2.3 (Pin_3), R7.2
- net +VDC: now also D3.1 (K); no longer R4.2
- net GND: now also D3.2 (A), D6.2 (A), R1.1, R16.1, RV1.1, SW2.1 (A)
- net Off42V: now also R4.2
- net at K1.A2, R6.2: now also RV1.2
- net at F1.2: now also Q1.2 (D); no longer K1.11
- new net: Q2.1 (G), R2.2, R3.1
- new net: F1.1, J1.3 (Pin_3), J2.3 (Pin_3)
- new net: D1.2 (A), Q1.1 (G), R1.2
- new net: J13.2 (Pin_2), R11.1
- new net: J13.3 (Pin_3), R11.2
- new net 5V_VOLTAGE: D6.1 (K), R15.1, R16.2
- new net OnGND: R3.2, SW2.2 (B)
- new net PC_REMOTE: J13.1 (Pin_1)
- new net SFT_IM: K1.11, Q2.2 (D), R7.2
Other:
- note removed: "tutaj dioda idealna!!!"
- moved on the sheet: C1, C10, C11, C12, C2, C3, C4, C5, C6, C7, C8, C9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

Commit message: temp_pms bloody FINISHED and ordered.
Parts:
- removed C6: 100nF, Capacitor_SMD:C_0402_1005Metric, symbol Device:C_Small
- added D10, D11: G2V4, LED_SMD:LED_0805_2012Metric, symbol Device:LED
- added D8, D9: B3V1, LED_SMD:LED_0805_2012Metric, symbol Device:LED
- added FB1: FerriteBead_Small, Resistor_SMD:R_0402_1005Metric_Pad0.72x0.64mm_HandSolder, symbol Device:FerriteBead_Small
- added H1, H2, H3: MountingHole_Pad, MountingHole:MountingHole_3.2mm_M3_Pad_Via, symbol Mechanical:MountingHole_Pad
- added R19, R20: 20, Resistor_SMD:R_0805_2012Metric, symbol Device:R
- added R21: 240, Resistor_SMD:R_0805_2012Metric, symbol Device:R
- added R22: 120, Resistor_SMD:R_0805_2012Metric, symbol Device:R
- added R23, R24, R25, R26: 10k, Resistor_SMD:R_0402_1005Metric, symbol Device:R_Small
- added R27: R, Resistor_SMD:R_0402_1005Metric, symbol Device:R
- J13: symbol Connector_Generic:Conn_01x03 -> Connector_Generic_MountingPin:Conn_01x03_MountingPin
Connections:
- net +3V3: now also FB1.1, R22.1, R23.2, R25.2; no longer C9.1, U2.9 (VDDA)
- net +5V: now also R21.1
- net +BATT: now also R27.2
- net 5V_VOLTAGE: now also U2.19 (PB1)
- net BUS_VOLTAGE: now also U2.18 (PB0)
- net CANSTBY: now also U2.33 (PA12)
- net GND: now also J13.MP (MountPin), D10.1 (K), D11.1 (K), D8.1 (K), D9.1 (K), H1.1, H2.1, H3.1, R24.1, R26.1
- net PC_REMOTE: now also U2.42 (PB6), R23.1, R24.2
- net RC: now also U2.14 (PA4), R25.1, R26.2
- net T2: now also U2.17 (PA7)
- net at D1.2 (A), Q1.1 (G), R1.2: now also R27.1
- net D1: now reaches U2.12 (PA2)
- net D1: now also R20.1
- net D2: now reaches U2.13 (PA3)
- net D2: now also R19.1
- new net: D11.2 (A), R22.2
- new net: D8.2 (A), R19.2
- new net: D10.2 (A), R21.2
- new net: C9.1, FB1.2, U2.9 (VDDA)
- new net: D9.2 (A), R20.2
Other:
- moved on the sheet: C4, C5, C7, C8, C9, R11
